Commit message: Add Gazebo room and differential drive control

File: src/ar01_description/urdf/ar01.urdf.xacro (robot description, xacro)
@@ -10,5 +10,11 @@
   <xacro:include filename="ar01_base.xacro"/>
   <xacro:include filename="ar01_sensors.xacro"/>
+  <xacro:include filename="ar01_ros2_control.xacro"/>
+  <xacro:arg name="use_sim" default="false"/>
+  <xacro:arg name="controller_config" default=""/>
   <xacro:ar01_base/>
   <xacro:ar01_sensors/>
+  <xacro:if value="$(arg use_sim)">
+    <xacro:ar01_ros2_control controller_config="$(arg controller_config)"/>
+  </xacro:if>
 </robot>

File: src/ar01_description/urdf/ar01_base.xacro (robot description, xacro)
@@ -31,4 +31,5 @@
     <link name="base_link">
       <visual>
+        <origin xyz="-0.025 0 0" rpy="0 0 0"/>
         <geometry>
           <box size="${body_length} ${body_width} ${body_height}"/>
@@ -37,4 +38,5 @@
       </visual>
       <collision>
+        <origin xyz="-0.025 0 0" rpy="0 0 0"/>
         <geometry>
           <box size="${body_length} ${body_width} ${body_height}"/>
@@ -42,5 +44,6 @@
       </collision>
       <inertial>
-        <origin xyz="0 0 0" rpy="0 0 0"/>
+        <!-- The drive axle is 25 mm forward of the chassis centre. -->
+        <origin xyz="-0.025 0 0" rpy="0 0 0"/>
         <mass value="${body_mass}"/>
         <!-- Solid box inertia about its centre. -->
@@ -54,5 +57,5 @@
       </inertial>
     </link>
-    <!-- base_link is at chassis centre; wheel centres are 50 mm above floor. -->
+    <!-- base_link is at the drive axle; wheel centres are 50 mm above floor. -->
     <joint name="base_footprint_joint" type="fixed">
       <parent link="base_footprint"/>
@@ -94,4 +97,5 @@
         <origin xyz="0 ${y} -0.050" rpy="0 0 0"/>
         <axis xyz="0 1 0"/>
+        <limit effort="20.0" velocity="20.0"/>
         <dynamics damping="0.1" friction="0.0"/>
       </joint>
@@ -130,4 +134,17 @@
       <origin xyz="-0.120 0 -0.075" rpy="0 0 0"/>
     </joint>
+    <!-- Contact parameters for the future Gazebo rigid-body simulation. -->
+    <gazebo reference="left_wheel_link">
+      <mu1>1.0</mu1>
+      <mu2>1.0</mu2>
+    </gazebo>
+    <gazebo reference="right_wheel_link">
+      <mu1>1.0</mu1>
+      <mu2>1.0</mu2>
+    </gazebo>
+    <gazebo reference="caster_link">
+      <mu1>0.001</mu1>
+      <mu2>0.001</mu2>
+    </gazebo>
   </xacro:macro>
 </robot>

File: src/ar01_description/urdf/ar01_ros2_control.xacro (robot description, xacro)
@@ -1,7 +1,33 @@
 <?xml version="1.0"?>
 <robot xmlns:xacro="http://www.ros.org/wiki/xacro">
-  <!--
-    Reserved for the ros2_control contract after description step 15.
-    This file is intentionally inactive in the geometry-only milestone.
-  -->
+  <xacro:macro name="ar01_ros2_control" params="controller_config">
+    <ros2_control name="GazeboSimSystem" type="system">
+      <hardware>
+        <plugin>gz_ros2_control/GazeboSimSystem</plugin>
+      </hardware>
+      <joint name="left_wheel_joint">
+        <command_interface name="velocity">
+          <param name="min">-20.0</param>
+          <param name="max">20.0</param>
+        </command_interface>
+        <state_interface name="position"/>
+        <state_interface name="velocity"/>
+      </joint>
+      <joint name="right_wheel_joint">
+        <command_interface name="velocity">
+          <param name="min">-20.0</param>
+          <param name="max">20.0</param>
+        </command_interface>
+        <state_interface name="position"/>
+        <state_interface name="velocity"/>
+      </joint>
+    </ros2_control>
+    <gazebo>
+      <plugin
+        filename="libgz_ros2_control-system.so"
+        name="gz_ros2_control::GazeboSimROS2ControlPlugin">
+        <parameters>${controller_config}</parameters>
+      </plugin>
+    </gazebo>
+  </xacro:macro>
 </robot>

File: src/ar01_description/urdf/ar01_sensors.xacro (robot description, xacro)
@@ -74,5 +74,5 @@
       <parent link="base_link"/>
       <child link="imu_link"/>
-      <origin xyz="0 0 0" rpy="0 0 0"/>
+      <origin xyz="-0.025 0 0" rpy="0 0 0"/>
     </joint>
   </xacro:macro>

Commit message: Add simulated LiDAR and IMU

File: src/ar01_description/urdf/ar01.urdf.xacro (robot description, xacro)
@@ -14,5 +14,5 @@
   <xacro:arg name="controller_config" default=""/>
   <xacro:ar01_base/>
-  <xacro:ar01_sensors/>
+  <xacro:ar01_sensors use_sim="$(arg use_sim)"/>
   <xacro:if value="$(arg use_sim)">
     <xacro:ar01_ros2_control controller_config="$(arg controller_config)"/>

File: src/ar01_description/urdf/ar01_sensors.xacro (robot description, xacro)
@@ -1,6 +1,6 @@
 <?xml version="1.0"?>
 <robot xmlns:xacro="http://www.ros.org/wiki/xacro">
-  <xacro:macro name="ar01_sensors">
-    <!-- Geometry placeholders only; sensor plugins are a later P0 step. -->
+  <xacro:macro name="ar01_sensors" params="use_sim">
+    <!-- Sensor geometry is shared by the physical model and the Gazebo plugins. -->
     <xacro:property name="lidar_radius" value="0.035"/>
     <xacro:property name="lidar_height" value="0.040"/>
@@ -76,4 +76,43 @@
       <origin xyz="-0.025 0 0" rpy="0 0 0"/>
     </joint>
+    <xacro:if value="${use_sim}">
+      <gazebo reference="lidar_link">
+        <sensor name="gpu_lidar" type="gpu_lidar">
+          <topic>/scan</topic>
+          <update_rate>10</update_rate>
+          <always_on>true</always_on>
+          <visualize>true</visualize>
+          <lidar>
+            <scan>
+              <horizontal>
+                <samples>720</samples>
+                <resolution>1</resolution>
+                <min_angle>${-pi}</min_angle>
+                <max_angle>${pi}</max_angle>
+              </horizontal>
+              <vertical>
+                <samples>1</samples>
+                <resolution>1</resolution>
+                <min_angle>0.0</min_angle>
+                <max_angle>0.0</max_angle>
+              </vertical>
+            </scan>
+            <range>
+              <min>0.10</min>
+              <max>12.0</max>
+              <resolution>0.01</resolution>
+            </range>
+          </lidar>
+        </sensor>
+      </gazebo>
+      <gazebo reference="imu_link">
+        <sensor name="imu_sensor" type="imu">
+          <topic>/imu/data</topic>
+          <update_rate>100</update_rate>
+          <always_on>true</always_on>
+          <visualize>false</visualize>
+        </sensor>
+      </gazebo>
+    </xacro:if>
   </xacro:macro>
 </robot>
